File: CM_V2-1.brd (EAGLE design)
At the start: 88.9 x 23.9 mm, 38 parts, among them M1 RN4870, SW1 147873-1, U1 OPA2333AIDR, U2 ADS1115IDGSR, U3 AT90USB1286-MUR

Commit message: Add files via upload
Parts:
- removed J3: (no value), SparkFun-Connectors:2X3_SMD
- added C10, C9: 0.1uF, SparkFun-Capacitors:0603
- added C8: 18pF, SparkFun-Capacitors:0603
- added J2: (no value), SparkFun-Connectors:2X3_SMD
- added R16: 10k, SparkFun-Resistors:0603
- added Y1: ECS-80-18-30B-AGN-TR, ECS-80-18-30B-AGN-TR:XTAL_ECS-80-18-30B-AGN-TR
- C7: value 0.1uF -> 18pF
- moved C7 17.4 mm to (36.8, 21.6), turned to 0 degrees
- moved R8 17.4 mm to (55.6, 16.8), turned to 270 degrees
- moved R13 14.9 mm to (52.6, 16.8), turned to 90 degrees
- moved R15 13.3 mm to (51.1, 16.8), turned to 270 degrees
- moved LED3 12.5 mm to (61.5, 22.4), turned to 180 degrees
- moved R6 11.2 mm to (57.1, 16.8), turned to 270 degrees
- moved R7 9.99 mm to (58.7, 16.8), turned to 270 degrees
- moved J1 8.82 mm to (68.3, 14.5), turned to 180 degrees
- moved LED2 6.27 mm to (66.3, 22.4)
- moved LED1 4.58 mm to (4.83, 22.4)
- moved LED4 3.59 mm to (71.6, 22.4)
- moved R5 3.44 mm to (8.26, 22.4), turned to 0 degrees
- moved SW1 2.62 mm to (54.4, 21.6), turned to 0 degrees
- moved R14 0.95 mm to (51.1, 13.5), turned to 270 degrees
- moved C2 0.38 mm to (29.1, 19.1)
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Connections:
- new net GND_2: U3.22
- new net N$25: C7.1, U3.23, Y1.1
- new net N$26: C8.1, U3.24, Y1.3
- new net N$27: R16.1, U2.2, U3.29
- new net VCC_2: U3.21
- net 3.3V: now also C10.1, C9.1, J2.2, R16.2, U3.52; no longer C7.1, J3.2, U3.21
- net GND: now also C10.2, C8.2, C9.2, J2.6, Y1.2, Y1.4; no longer J3.6, U3.22
- net N$21: now also J2.4; no longer J3.4
- net N$22: now also J2.1; no longer J3.1
- net N$23: now also J2.3; no longer J3.3
- net N$24: now also J2.5; no longer J3.5
- net VCC: no longer U3.52
Routing:
- net VCC: track 21.8 -> 84.1 mm, vias 0 -> 2
- net N$10: track 0.00 -> 49.3 mm, vias 0 -> 2
- net N$9: track 0.00 -> 47.5 mm, vias 0 -> 2
- net N$21: track 0.00 -> 43.4 mm, vias 0 -> 2
- net N$22: track 0.00 -> 41.7 mm, vias 0 -> 2
- net N$24: track 0.00 -> 37.6 mm, vias 0 -> 3
- net N$23: track 0.00 -> 36.1 mm, vias 0 -> 2
- net N$18: track 0.00 -> 33.5 mm, vias 0 -> 2
- net N$20: track 0.00 -> 29.0 mm, vias 0 -> 2
- net N$19: track 0.00 -> 26.1 mm, vias 0 -> 2
- net N$17: track 0.00 -> 22.7 mm, vias 0 -> 2
- net N$27: track 0.00 -> 19.4 mm, vias 0 -> 3
- net N$25: track 0.00 -> 15.9 mm, vias 0 -> 2
- net GND: track 52.0 -> 66.8 mm, vias 7 -> 11
- net N$15: track 0.00 -> 14.9 mm, vias 0 -> 2
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- added copper zone on layer 1, net GND
Other:
- board size 88.9 x 23.9 mm -> 88.9 x 23.6 mm
- board text added: "GND"
- board text added: "Mode"
- board text added: "Power"
- board text added: "Status 1"
- board text added: "Status 2"
- board text added: "VCC"

Commit message: Add files via upload
Parts:
- added C11, C12: 0.1uF, SparkFun-Capacitors:0603
- added R17, R18: 10k, SparkFun-Resistors:0603
- C4: value 22nF -> 0.1uF
- C6: value 0.22uF -> 22nF
- C7: value 18pF -> 0.22uF
- C9: value 0.1uF -> 18pF
- J1: value (none) -> 1771033; device SparkFun-Connectors:JST-2-SMD-VERT -> 1771033:PHOENIX_1771033
- LED2, LED3: value GRN -> RED
- R13: value 10k -> 150k
- R14: value 10k -> 11k
- moved J1 64.6 mm to (4.06, 7.62), flipped to the bottom, turned to 90 degrees
- moved C3 24.9 mm to (73.7, 15.0), turned to 90 degrees
- moved C10 14.7 mm to (49.5, 9.60), turned to 270 degrees
- moved C7 14.5 mm to (40.6, 7.62)
- moved C9 13.4 mm to (36.8, 14.0), turned to 180 degrees
- moved C4 10.6 mm to (50.6, 5.46), turned to 270 degrees
- moved R14 9.71 mm to (60.2, 16.8)
- moved R13 9.14 mm to (61.7, 16.8)
- moved C8 7.62 mm to (36.8, 21.6), turned to 0 degrees
- moved R16 4.48 mm to (51.1, 13.5)
- moved C5 3.05 mm to (40.6, 9.14), turned to 180 degrees
- moved R15 1.52 mm to (52.6, 16.8), turned to 90 degrees
- moved C6 1.52 mm to (40.6, 6.10)
Connections:
- removed net AVCC: U3.64
- removed net GND_2: U3.22
- removed net GND_3: U3.53
- removed net VCC_2: U3.21
- new net N$30: R13.1, R14.1, U2.6
- net 3.3V: now also C11.1, C12.1, C4.1, R15.1, R16.1, R17.2, R18.2, U3.21, U3.64; no longer C9.1, R13.1, R14.1, R15.2, R16.2
- net GND: now also C11.2, C12.2, C5.2, C6.1, R14.2, U2.7, U3.22, U3.53, U3.65; no longer C5.1, C7.2, J1.GND
- net N$1: now also C5.1, C7.1; no longer C4.1, C6.1
- net N$10: now also J1.1
- net N$19: now also U3.31
- net N$20: now also U3.32
- net N$24: now also M1.21, R18.1; no longer R15.1
- net N$25: now also C8.1; no longer C7.1
- net N$26: now also C9.1; no longer C8.1
- net N$27: now also R17.1, U3.19; no longer R16.1, U3.29
- net N$3: now also R15.2; no longer R13.2
- net N$4: now also R16.2; no longer R14.2
- net N$7: now also C7.2; no longer C5.2
- net N$9: now also J1.2
- net VCC: now also J1.3, R13.2; no longer J1.VCC
Routing:
- net N$20: track 29.0 -> 74.4 mm, vias 2 -> 3
- net N$9: track 47.5 -> 92.3 mm
- net N$19: track 26.1 -> 66.8 mm, vias 2 -> 3
- net N$10: track 49.3 -> 89.9 mm
- net GND: track 66.8 -> 94.9 mm, vias 11 -> 13
- net N$30: track 0.00 -> 25.9 mm, vias 0 -> 2
- net N$24: track 37.6 -> 60.4 mm, vias 3 -> 4
- net N$27: track 19.4 -> 25.1 mm
- net 3.3V: track 29.1 -> 34.2 mm, vias 11 -> 12
- net VCC: track 84.1 -> 88.6 mm
Other:
- board text added: "Electric Current Monitor v2.0 Oct 2019"
- board text added: "ISP"
- board text added: "RX"
- board text added: "TX"
- board text removed: "GND"
