File: CM_V2-1.sch (EAGLE design)
At the start: 38 parts, among them M1 RN4870, SW1 147873-1, U1 OPA2333AIDR, U2 ADS1115IDGSR, U3 AT90USB1286-MUR

Commit message: Add files via upload
Parts:
- added C10, C9: 0.1uF, SparkFun-Capacitors:0.1UF-0603-25V-5%
- added C8: 18pF, SparkFun-Capacitors:18PF-0603-50V-5%
- added R16: 10k, SparkFun-Resistors:10KOHM-0603-1/10W-1%
- added Y1: ECS-80-18-30B-AGN-TR, ECS-80-18-30B-AGN-TR:ECS-80-18-30B-AGN-TR
- C7: value 0.1uF -> 18pF; device SparkFun-Capacitors:0.1UF-0603-25V-5% -> SparkFun-Capacitors:18PF-0603-50V-5%
- renumbered J3 to J2
Connections:
- new net N$25: C7.1, U3.XTAL2, Y1.IN/OUT
- new net N$26: C8.1, U3.XTAL1, Y1.OUT/IN
- new net N$27: R16.1, U2.ALERT/RDY, U3.PD4
- net 3.3V: now also C10.1, C9.1, R16.2, U3.VCC; no longer C7.1, U3.VCC_2
- net GND: now also C10.2, C8.2, C9.2, U3.GND, Y1.GND; no longer U3.GND_2
Other:
- note added: "LED0: Provides indication whether the module is in ON/OFF mode"
- note added: "Power Indicator"
- note added: "Pull up resistors"
- note added: "Reset switch"
- note added: "Status 1"
- note added: "Status 2"
- moved on the sheet: C7

Commit message: Add files via upload
Parts:
- added C11, C12: 0.1uF, SparkFun-Capacitors:0.1UF-0603-25V-5%
- added R17, R18: 10k, SparkFun-Resistors:10KOHM-0603-1/10W-1%
- C3: device SparkFun-Capacitors:0.1UF-0603-25V-(+80/-20%) -> SparkFun-Capacitors:0.1UF-0603-25V-5%
- C4: value 22nF -> 0.1uF; device SparkFun-Capacitors:22NF/22,000PF-0603-50V-10% -> SparkFun-Capacitors:0.1UF-0603-25V-(+80/-20%)
- C6: value 0.22uF -> 22nF; device SparkFun-Capacitors:0.22UF-0603-25V-10% -> SparkFun-Capacitors:22NF/22,000PF-0603-50V-10%
- C7: value 18pF -> 0.22uF; device SparkFun-Capacitors:18PF-0603-50V-5% -> SparkFun-Capacitors:0.22UF-0603-25V-10%
- C9: value 0.1uF -> 18pF; device SparkFun-Capacitors:0.1UF-0603-25V-5% -> SparkFun-Capacitors:18PF-0603-50V-5%
- J1: value (none) -> 1771033; device SparkFun-Connectors:CONN_024UCON-15767 -> 1771033:1771033
- LED2, LED3: value GRN -> RED
- R13: value 10k -> 150k; device SparkFun-Resistors:10KOHM-0603-1/10W-1% -> SparkFun-Resistors:150KOHM-0603-1/10W-1%
- R14: value 10k -> 11k; device SparkFun-Resistors:10KOHM-0603-1/10W-1% -> SparkFun-Resistors:RESISTOR0603
Connections:
- new net N$30: R13.1, R14.1, U2.AIN2
- net 3.3V: now also C11.1, C12.1, C4.1, R15.1, R16.1, R17.2, R18.2, U3.AVCC, U3.VCC_2; no longer C9.1, R13.1, R14.1, R15.2, R16.2
- net GND: now also C11.2, C12.2, C5.2, C6.1, R14.2, U2.AIN3, U3.EPAD, U3.GND_2, U3.GND_3; no longer C5.1, C7.2, J1.1
- net N$1: now also C5.1, C7.1; no longer C4.1, C6.1
- net N$10: now also J1.1
- net N$19: now also U3.PD6
- net N$20: now also U3.PD7
- net N$24: now also M1.R\S\T\@1, R18.1; no longer R15.1
- net N$25: now also C8.1; no longer C7.1
- net N$26: now also C9.1; no longer C8.1
- net N$27: now also R17.1, U3.PE5; no longer R16.1, U3.PD4
- net N$3: now also R15.2; no longer R13.2
- net N$4: now also R16.2; no longer R14.2
- net N$7: now also C7.2; no longer C5.2
- net N$9: now also J1.2
- net VCC: now also J1.3, R13.2; no longer J1.2
Other:
- moved on the sheet: C10, C3, C4, C5, C6, C7, C8, C9, R13, R14, R15, R16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
